File: hw/101001-powersupply/display.kicad_sch (KiCad schematic)
At the start: 1 part, among them J601 BM24-40DS

Commit message: Progress on board design
Connections:
- net EXT8 is gone; now on net GND: J601.8 (Pin_8)
- net GND: now also J601.28 (Pin_28); no longer J601.10 (Pin_10), J601.18 (Pin_18), J601.30 (Pin_30), J601.6 (Pin_6)
- net SCL: now also J601.32 (Pin_32); no longer J601.28 (Pin_28)
- net SDA: now also J601.30 (Pin_30); no longer J601.32 (Pin_32)
- new net EXT10: J601.10 (Pin_10)
- new net EXT18: J601.18 (Pin_18)
- new net EXT6: J601.6 (Pin_6)
Other:
- company: (none) -> Sarif
- title: (none) -> Variable USB power supply
