File: hw/101001-powersupply/101001-powersupply.kicad_sch (KiCad schematic)
At the start: 17 parts, among them J101 GT-USB-7010ASV, J102 GT-USB-7010ASV, J103 2604-1102

Commit message: Progress on board design
Parts:
- J102: value GT-USB-7010ASV -> GT-USB-7051A; footprint Connector_USB:USB_C_Receptacle_G-Switch_GT-USB-7010ASV -> Connector_USB:USB_C_Receptacle_G-Switch_GT-USB-7051x; LCSC C2988369 -> C2843970
Other:
- sheet Display ports: added EXT10, EXT18, EXT6; removed EXT8
- sheet Microcontroller ports: added GPIO0, GPIO1; removed none
- company: (none) -> Sarif
- title: (none) -> Variable USB power supply
Changed lines of the file:
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@@
 	(generator_version "8.0")
 	(paper "A4")
+	(title_block
+		(title "Variable USB power supply")
+		(date "2024-04-23")
+		(rev "1")
+		(company "Sarif")
+	)
 	(junction
 		(at 234.95 130.81)
@@
 	(wire
 		(pts
+			(xy 63.5 144.78) (xy 92.71 144.78)
+		)
+		(stroke
+			(width 0)
+			(type default)
+		)
+	)
+	(wire
+		(pts
 			(xy 168.91 58.42) (xy 168.91 60.96)
 		)
@@
 	(wire
 		(pts
+			(xy 63.5 147.32) (xy 92.71 147.32)
+		)
+		(stroke
+			(width 0)
+			(type default)
+		)
+	)
+	(wire
+		(pts
 			(xy 252.73 105.41) (xy 252.73 107.95)
 		)
@@
 		(dnp no)
 		(fields_autoplaced yes)
-		(property "Reference" "#PWR0109"
+		(property "Reference" "#PWR0104"
 			(at 203.2 88.9 0)
 			(effects
@@
 			(project "101001-powersupply"
 				(path "/5b6c9e65-6d2e-4a49-a6e0-6edf7b37266c"
-					(reference "#PWR0109")
+					(reference "#PWR0104")
 					(unit 1)
 				)
@@
 		(dnp no)
 		(fields_autoplaced yes)
-		(property "Reference" "#PWR0108"
+		(property "Reference" "#PWR0101"
 			(at 167.64 139.7 0)
 			(effects
@@
 			(project "101001-powersupply"
 				(path "/5b6c9e65-6d2e-4a49-a6e0-6edf7b37266c"
-					(reference "#PWR0108")
+					(reference "#PWR0101")
 					(unit 1)
 				)
@@
 			)
 		)
-		(property "Value" "GT-USB-7010ASV"
+		(property "Value" "GT-USB-7051A"
 			(at 234.95 82.55 0)
 			(effects
@@
 			)
 		)
-		(property "Footprint" "Connector_USB:USB_C_Receptacle_G-Switch_GT-USB-7010ASV"
+		(property "Footprint" "Connector_USB:USB_C_Receptacle_G-Switch_GT-USB-7051x"
 			(at 238.76 102.87 0)
 			(effects
@@
 			)
 		)
-		(property "LCSC" "C2988369"
+		(property "LCSC" "C2843970"
 			(at 234.95 102.87 0)
 			(effects
@@
 		(dnp no)
 		(fields_autoplaced yes)
-		(property "Reference" "#PWR0103"
+		(property "Reference" "#PWR0105"
 			(at 208.28 39.37 0)
 			(effects
@@
 			(project "101001-powersupply"
 				(path "/5b6c9e65-6d2e-4a49-a6e0-6edf7b37266c"
-					(reference "#PWR0103")
+					(reference "#PWR0105")
 					(unit 1)
 				)
@@
 		(dnp no)
 		(fields_autoplaced yes)
-		(property "Reference" "#PWR0111"
+		(property "Reference" "#PWR0107"
 			(at 232.41 41.91 0)
 			(effects
@@
 			(project "101001-powersupply"
 				(path "/5b6c9e65-6d2e-4a49-a6e0-6edf7b37266c"
-					(reference "#PWR0111")
+					(reference "#PWR0107")
 					(unit 1)
 				)
@@
 		(dnp no)
 		(fields_autoplaced yes)
-		(property "Reference" "#PWR0112"
+		(property "Reference" "#PWR0108"
 			(at 232.41 62.23 0)
 			(effects
@@
 			(project "101001-powersupply"
 				(path "/5b6c9e65-6d2e-4a49-a6e0-6edf7b37266c"
-					(reference "#PWR0112")
+					(reference "#PWR0108")
 					(unit 1)
 				)
@@
 		(dnp no)
 		(fields_autoplaced yes)
-		(property "Reference" "#PWR0113"
+		(property "Reference" "#PWR0109"
 			(at 261.62 88.9 0)
 			(effects
@@
 			(project "101001-powersupply"
 				(path "/5b6c9e65-6d2e-4a49-a6e0-6edf7b37266c"
-					(reference "#PWR0113")
+					(reference "#PWR0109")
 					(unit 1)
 				)
@@
 		(dnp no)
 		(fields_autoplaced yes)
-		(property "Reference" "#FLG0103"
+		(property "Reference" "#FLG0102"
 			(at 199.39 33.655 0)
 			(effects
@@
 			(project "101001-powersupply"
 				(path "/5b6c9e65-6d2e-4a49-a6e0-6edf7b37266c"
-					(reference "#FLG0103")
+					(reference "#FLG0102")
 					(unit 1)
 				)
@@
 		(dnp no)
 		(fields_autoplaced yes)
-		(property "Reference" "#PWR0110"
+		(property "Reference" "#PWR0106"
 			(at 227.33 139.7 0)
 			(effects
@@
 			(project "101001-powersupply"
 				(path "/5b6c9e65-6d2e-4a49-a6e0-6edf7b37266c"
-					(reference "#PWR0110")
+					(reference "#PWR0106")
 					(unit 1)
 				)
@@
 		(dnp no)
 		(fields_autoplaced yes)
-		(property "Reference" "#PWR0101"
+		(property "Reference" "#PWR0102"
 			(at 168.91 50.8 0)
 			(effects
@@
 			(project "101001-powersupply"
 				(path "/5b6c9e65-6d2e-4a49-a6e0-6edf7b37266c"
-					(reference "#PWR0101")
+					(reference "#PWR0102")
 					(unit 1)
 				)
@@
 		(dnp no)
 		(fields_autoplaced yes)
-		(property "Reference" "#PWR0102"
+		(property "Reference" "#PWR0103"
 			(at 168.91 62.23 0)
 			(effects
@@
 			(project "101001-powersupply"
 				(path "/5b6c9e65-6d2e-4a49-a6e0-6edf7b37266c"
-					(reference "#PWR0102")
+					(reference "#PWR0103")
 					(unit 1)
 				)
@@
 		(dnp no)
 		(fields_autoplaced yes)
-		(property "Reference" "#FLG0102"
+		(property "Reference" "#FLG0103"
 			(at 252.73 83.185 0)
 			(effects
@@
 			(project "101001-powersupply"
 				(path "/5b6c9e65-6d2e-4a49-a6e0-6edf7b37266c"
-					(reference "#FLG0102")
+					(reference "#FLG0103")
 					(unit 1)
 				)
@@
 		)
 		(pin "GPIO2" bidirectional
-			(at 92.71 134.62 180)
+			(at 92.71 139.7 180)
 			(effects
 				(font
@@
 		)
 		(pin "GPIO9" bidirectional
-			(at 92.71 142.24 180)
+			(at 92.71 147.32 180)
 			(effects
 				(font
@@
 		)
 		(pin "GPIO6" bidirectional
-			(at 92.71 137.16 180)
+			(at 92.71 142.24 180)
 			(effects
 				(font
@@
 		)
 		(pin "GPIO8" bidirectional
-			(at 92.71 139.7 180)
+			(at 92.71 144.78 180)
+			(effects
+				(font
+					(size 1.27 1.27)
+				)
+				(justify left)
+			)
+		)
+		(pin "GPIO0" bidirectional
+			(at 92.71 134.62 180)
+			(effects
+				(font
+					(size 1.27 1.27)
+				)
+				(justify left)
+			)
+		)
+		(pin "GPIO1" bidirectional
+			(at 92.71 137.16 180)
 			(effects
 				(font
@@
 			)
 		)
+		(pin "SCL" bidirectional
+			(at 63.5 123.19 0)
+			(effects
+				(font
+					(size 1.27 1.27)
+				)
+				(justify right)
+			)
+		)
+		(pin "SDA" bidirectional
+			(at 63.5 125.73 0)
+			(effects
+				(font
+					(size 1.27 1.27)
+				)
+				(justify right)
+			)
+		)
 		(pin "EXT12" bidirectional
-			(at 63.5 139.7 0)
+			(at 63.5 142.24 0)
 			(effects
 				(font
@@
 			)
 		)
-		(pin "EXT4" bidirectional
-			(at 63.5 134.62 0)
+		(pin "EXT10" bidirectional
+			(at 63.5 139.7 0)
 			(effects
 				(font
@@
 			)
 		)
-		(pin "EXT8" bidirectional
-			(at 63.5 137.16 0)
+		(pin "EXT4" bidirectional
+			(at 63.5 134.62 0)
 			(effects
 				(font
@@
 			)
 		)
-		(pin "EXT16" bidirectional
-			(at 63.5 142.24 0)
+		(pin "EXT6" bidirectional
+			(at 63.5 137.16 0)
 			(effects
 				(font
@@
 			)
 		)
-		(pin "SCL" bidirectional
-			(at 63.5 123.19 0)
+		(pin "EXT18" bidirectional
+			(at 63.5 147.32 0)
 			(effects
 				(font
@@
 			)
 		)
-		(pin "SDA" bidirectional
-			(at 63.5 125.73 0)
+		(pin "EXT16" bidirectional
+			(at 63.5 144.78 0)
 			(effects
 				(font

Commit message: Finalized board design
Other:
- sheet Interal powersupply renamed Internal powersupply
Changed lines of the file:
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@@
 			(color 0 0 0 0.0000)
 		)
-		(property "Sheetname" "Interal powersupply"
+		(property "Sheetname" "Internal powersupply"
 			(at 25.4 37.3884 0)
 			(effects

Commit message: Hardware improvements
Parts:
- added R101, R102: 1kOhm, Resistor_SMD:R_0402_1005Metric, symbol Device:R
Connections:
- net GND: now also R101.1, R102.1
- net VPROG: now also R102.2
- net VSUPPLY: now also R101.2
Other:
- note added: "1mA leakage reverse-bias"
- note added: "Power rail pull-downs"
- note added: "to measure when not biased"
- moved on the sheet: D101, D102, D103, D104, D105, D106, D107, D108, D109, F101, J101, J102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
