File: hw/101001-powersupply/psu-external.kicad_sch (KiCad schematic)
At the start: 30 parts, among them Q301 2N7002, Q302 2N7002, U301 TPS55289RYQR

Commit message: Progress on board design
Connections:
- net VOUT_MEAS renamed VOUT_ISN
Other:
- note added: "2V-20V 4A"
- note added: "5V-20V 0.5A-3A"
- note added: "AGND nettie near VCC capacitor ground"
- note added: "As per page 41, 10.1 Layout Guidelines"
- note added: "Enable and UVLO circuit with correct boot bias"
- note added: "External buck-boost powersupply"
- note added: "I2C address: 0x74"
- note added: "with variable voltage & current limiting"
- company: (none) -> Sarif
- title: (none) -> Variable USB power supply
- moved on the sheet: C302, C303, C304, C305, C306, C307, C308, C309, C310, C311, C312, C313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

Commit message: Finalized board design
Parts:
- added C317: (no value), Capacitor_SMD:C_0402_1005Metric, symbol Device:C
- added D301: KT-0603G Emerald, LED_SMD:LED_0603_1608Metric, symbol Device:LED
- added Q303: 2N7002, Package_TO_SOT_SMD:SOT-23, symbol Transistor_FET:2N7002
- added R310, R311: 1kOhm, Resistor_SMD:R_0402_1005Metric, symbol Device:R
Connections:
- net GND: now also Q303.2 (S)
- net VOUT_DIRECT: now also C317.1, Q303.1 (G)
- net VOUT_ISN: now also C317.2
- new net LED_OD: D301.1 (K), Q303.3 (D)
- new net LED_VDD: D301.2 (A), R310.1, R311.2
- new net VDD: R310.2, R311.1
Other:
- note added: "Indicator LED"
- note added: "Vf=2.75V I=1mA"

Commit message: Fixed Ccomp
Parts:
- C317: value (none) -> ~
Changed lines of the file:
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@@
 			)
 		)
-		(property "Value" ""
+		(property "Value" "~"
 			(at 261.62 93.98 90)
 			(effects

Commit message: Hardware improvements
Parts:
- R304: value 887kOhm -> 100kOhm; LCSC C137930 -> C25741
- R305: now not fitted; now left out of the parts list
Other:
- note removed: "0.5V-2V"
Changed lines of the file:
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@@
 		)
 	)
-	(text "0.5V-2V"
+	(text "5V-20V"
 		(exclude_from_sim no)
 		(at 73.66 123.19 0)
@@
 			)
 		)
-		(property "Value" "887kOhm"
+		(property "Value" "100kOhm"
 			(at 78.74 111.76 90)
 			(effects
@@
 			)
 		)
-		(property "LCSC" "C137930"
+		(property "LCSC" "C25741"
 			(at 80.01 107.95 0)
 			(effects
@@
 		(unit 1)
 		(exclude_from_sim no)
-		(in_bom yes)
-		(on_board yes)
-		(dnp no)
+		(in_bom no)
+		(on_board yes)
+		(dnp yes)
 		(property "Reference" "R305"
 			(at 85.09 146.05 0)
