File: hw/101001-powersupply/usb-pd.kicad_sch (KiCad schematic)
At the start: 8 parts, among them U501 STUSB4500QTR

Commit message: Progress on board design
Other:
- company: (none) -> Sarif
- title: (none) -> Variable USB power supply
Changed lines of the file:
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@@
 	(generator_version "8.0")
 	(paper "A4")
+	(title_block
+		(title "Variable USB power supply")
+		(date "2024-04-23")
+		(rev "1")
+		(company "Sarif")
+	)
 	(junction
 		(at 143.51 54.61)

Commit message: Finalized board design
Parts:
- added D501: KT-0603R Red, LED_SMD:LED_0603_1608Metric, symbol Device:LED
- added R505: 1kOhm, Resistor_SMD:R_0402_1005Metric, symbol Device:R
Connections:
- net LED_OD: now reaches U501.15 (GPIO)
- net LED_OD: now also D501.1 (K)
- new net LED_VDD: D501.2 (A), R505.1
- new net VDD: R505.2
- no-connect marks 7 -> 6
Other:
- note added: "Vf=2.05V I=1mA"

Commit message: Hardware improvements
Parts:
- added R506: 0ohm, Resistor_SMD:R_0402_1005Metric, symbol Device:R
Connections:
- net GND: no longer U501.22 (VSYS)
- net VDD: now also R506.1
- new net PD_VSYS: R506.2, U501.22 (VSYS)
